Commit message: Initial Commit for Roboshield Demo Branch

File: ur_e_description/urdf/ur10e_joint_limited_robot.urdf.xacro (robot description, xacro)
@@ -15,7 +15,7 @@
 		 wrist_3_lower_limit="${-pi}" wrist_3_upper_limit="${pi}"
 />
-  <link name="world" />
-  <joint name="world_joint" type="fixed">
-    <parent link="world" />
+  <link name="robot_base" />
+  <joint name="robot_base_joint" type="fixed">
+    <parent link="robot_base" />
     <child link = "base_link" />
     <origin xyz="0.0 0.0 0.0" rpy="0.0 0.0 0.0" />

File: ur_e_description/urdf/ur10e_robot.urdf.xacro (robot description, xacro)
@@ -8,7 +8,7 @@
   <!-- arm -->
   <xacro:ur10e_robot prefix="" joint_limited="false"/>
-  <link name="world" />
-  <joint name="world_joint" type="fixed">
-    <parent link="world" />
+  <link name="robot_base" />
+  <joint name="robot_base_joint" type="fixed">
+    <parent link="robot_base" />
     <child link = "base_link" />
     <origin xyz="0.0 0.0 0.0" rpy="0.0 0.0 0.0" />
